File: schematics/board/MA_board_1.brd (EAGLE design)
At the start: 68 x 75.2 mm, 69 parts, among them IC1 STM32F401RCT6

Commit message: новая версия первой платы нижнего модуля
Parts:
- removed R1: 10k, rcl:R0603
- added C10: 10nF, rcl:C0603
- added C11: 4.7uf, rcl:C0603
- added C12, C13: 100nF, rcl:C0603
- added C8: 1nF, rcl:C0603
- added C9: 100nf, rcl:C0603
- added Q24: Q24, CanCubeSat:Q24
- R17: value 100R -> 191k
- U$1: value LIS3MDL_CJMCU -> LIS3MDL-CJMCUБез_отв._зеркальный; device NEON-BLADE-2023:LIS3MDL-GY_CGMSU -> NEON-BLADE-2023:LIS3MDL-CGMSU-NB2023
- U$2: value LSM6DS3-GY -> LSM6DS3-GY-NB2023; device NEON-BLADE-2023:LSM6DS3-GY -> NEON-BLADE-2023:LSM6DS3-GY-NB2023
- moved R33 180.9 mm to (-38.0, 108.0), turned to 180 degrees
- moved R34 168.8 mm to (-38.0, 101.0), turned to 180 degrees
- moved U$19 166.5 mm to (-37.5, 105.0)
- moved R24 165.4 mm to (28.9, 94.0)
- moved R29 164.3 mm to (27.4, 102.5)
- moved R25 160.1 mm to (13.6, 97.6)
- moved R26 160.1 mm to (13.7, 100.1)
- moved R27 160.1 mm to (17.5, 99.6)
- moved R28 160.1 mm to (16.1, 103.5)
- moved U$15 160.1 mm to (12.8, 104.0)
- moved R32 152.9 mm to (-37.0, 96.6)
- moved U$13 152.8 mm to (18.6, 90.8), turned to 270 degrees
- moved U$17 151.9 mm to (25.4, 88.0), turned to 90 degrees
- moved R10 151.1 mm to (56.8, 23.5)
- moved R31 149.6 mm to (48.0, 59.0), turned to 90 degrees
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Connections:
- net BUTTON_DA_UP renamed FEEDBACK_DA
- net DA_DOWN_ON renamed BOTTON_DA_DOWN
- net DA_UP_ON renamed BOTTON_DA_UP
- net PAR_DOWN_ON renamed BOTTON_PAR_DOWN
- net PAR_UP_ON renamed BOTTON_PAR_UP
- net SKIRT_CLOSE_ON renamed BOTTON_SKIRT_CLOSE
- net SKIRT_OPEN_ON renamed BOTTON_SKIRT_OPEN
- removed net BUTTON_DA_DOWN: JP1.2, U$8.P$4
- removed net BUTTON_SKIRT_CLOSE: JP1.3, JP7.6
- removed net BUTTON_SKIRT_OPEN: JP1.5, JP7.5
- removed net N$35: IC1.7, R1.2
- new net FEEDBACK_SKIRT: C12.2, JP1.3, JP7.6
- new net FEEDBACK_SKIRT1: C13.2
- new net N$10: C8.2, Q24.P$3
- new net N$12: C11.1, IC1.30
- new net NRST: C9.2, IC1.7, JP1.5
- new net TCXO: C8.1, IC1.5
- net 3V3: now also C10.2, Q24.P$4; no longer R1.1
- net GND: now also C10.1, C11.2, C12.1, C13.1, C9.1, Q24.P$2
Routing:
- net N$5: track 5.46 -> 75.8 mm
- net N$9: track 15.7 -> 81.2 mm
- net GND: track 29.4 -> 81.4 mm
- net 3V3: track 0.00 -> 41.2 mm
- net SDIO_DAT2: track 0.00 -> 17.8 mm
- net 5V: track 17.8 -> 35.2 mm, vias 2 -> 4
- net SDIO_DAT3: track 0.00 -> 16.2 mm
- net SDIO_CMD: track 0.00 -> 15.8 mm
- net SDIO_DAT0: track 0.00 -> 13.2 mm
- net SDIO_DAT1: track 0.00 -> 13.0 mm
- net BOTTON_DA_UP: track 0.00 -> 11.8 mm
- net BOTTON_DA_DOWN: track 0.00 -> 11.7 mm
- net N$2: track 0.00 -> 9.90 mm
- net N$20: track 0.00 -> 4.21 mm
- net N$8: track 0.00 -> 4.00 mm
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Other:
- outline, holes or cut-outs redrawn

Commit message: немного продвинул работу над платой (Прмгите)
Parts:
- removed C12, C13: 100nF, rcl:C0603
- added R1, R35: 10k, rcl:R0603
- moved LED2 121.3 mm to (62.5, 44.0), turned to 180 degrees
- moved R4 120.5 mm to (59.0, 43.3)
- moved C5 113.5 mm to (59.0, 50.0)
- moved C3 112.6 mm to (54.5, 39.0), turned to 90 degrees
- moved R32 110.8 mm to (59.0, 41.2)
- moved C2 107.8 mm to (56.6, 37.5)
- moved C6 107.6 mm to (54.2, 57.0), turned to 90 degrees
- moved R6 104.2 mm to (46.5, 39.0), turned to 270 degrees
- moved LED1 96.1 mm to (42.0, 56.5), turned to 0 degrees
- moved C1 95.0 mm to (41.0, 44.5), turned to 180 degrees
- moved R5 94.9 mm to (41.0, 46.6)
- moved R3 93.9 mm to (39.5, 56.5), turned to 90 degrees
- moved C4 89.5 mm to (44.5, 56.0), turned to 90 degrees
- moved R33 88.2 mm to (22.2, 43.5), turned to 270 degrees
- moved U$19 83.3 mm to (17.5, 42.5), turned to 90 degrees
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Connections:
- removed net FEEDBACK_SKIRT1: C13.2
- new net NRF_IRQ: JP7.5
- net 3V3: now also R1.2, R35.1
- net CE_NRF: no longer IC1.2
- net CS_NRF: no longer IC1.3
- net FEEDBACK_DA: now also R35.2
- net FEEDBACK_SKIRT: now also R1.1; no longer C12.2
- net GND: now also U$8.P$4; no longer C12.1, C13.1
- net LED: now also IC1.2
- net MOSI: now also JP6.3; no longer JP6.1
- net SCK: now also JP6.1; no longer JP6.3
Routing:
- net SDA: track 0.00 -> 95.0 mm, vias 0 -> 5
- net SCL: track 0.00 -> 94.2 mm, vias 0 -> 2
- net MISO: track 0.00 -> 92.1 mm, vias 0 -> 1
- net MOSI: track 0.00 -> 84.0 mm, vias 0 -> 1
- net NRST: track 0.00 -> 66.5 mm, vias 0 -> 2
- net SCK: track 0.00 -> 58.1 mm
- net 3V3: track 41.2 -> 82.8 mm
- net SVC: track 0.00 -> 39.2 mm, vias 0 -> 2
- net GPS_RX: track 0.00 -> 37.3 mm, vias 0 -> 3
- net DBG_RX: track 0.00 -> 36.3 mm, vias 0 -> 1
- net DBG_TX: track 0.00 -> 36.0 mm, vias 0 -> 1
- net SVD: track 0.00 -> 34.2 mm, vias 0 -> 2
- net GPS_TX: track 0.00 -> 34.2 mm, vias 0 -> 3
- net SDIO_DAT1: track 13.0 -> 41.5 mm, vias 0 -> 2
- net SDIO_DAT2: track 17.8 -> 45.5 mm
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Other:
- board size 68 x 75.2 mm -> 68.5 x 75.2 mm

Commit message: Проверил платы. Исправил некоторые ошибки
Routing:
- net 3V3: track 82.8 -> 82.2 mm
Changed lines of the file:
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@@
 <contactref element="R1" pad="2"/>
 <contactref element="R35" pad="1"/>
-<wire x1="62.5" y1="44.75" x2="63.625" y2="44.75" width="0.2" layer="1"/>
-<wire x1="63.625" y1="44.75" x2="63.625" y2="46.65" width="0.2" layer="1"/>
 <wire x1="44.762" y1="43.75" x2="42.50695" y2="43.75" width="0.2" layer="1"/>
 <wire x1="42.50695" y1="43.75" x2="42.50455" y2="43.7476" width="0.2" layer="1"/>
@@
 <wire x1="56.6" y1="38.9" x2="58.15" y2="40.45" width="0.2" layer="1"/>
 <wire x1="58.15" y1="40.45" x2="58.15" y2="41.18" width="0.2" layer="1"/>
-<wire x1="47.01440625" y1="52.2481" x2="52.98559375" y2="52.2481" width="0.2" layer="1"/>
-<wire x1="53.25" y1="53.238" x2="53.25" y2="52.51250625" width="0.2" layer="1"/>
-<wire x1="53.25" y1="52.51250625" x2="53.118746875" y2="52.381253125" width="0.2" layer="1"/>
-<wire x1="53.118746875" y1="52.381253125" x2="52.98559375" y2="52.2481" width="0.2" layer="1"/>
 <wire x1="46.75" y1="53.238" x2="46.75" y2="52.51250625" width="0.2" layer="1"/>
 <wire x1="46.75" y1="52.51250625" x2="47.01440625" y2="52.2481" width="0.2" layer="1"/>
-<wire x1="53.118746875" y1="52.381253125" x2="55.2481" y2="50.2519" width="0.2" layer="1"/>
-<wire x1="55.2481" y1="50.2519" x2="55.2481" y2="50.01440625" width="0.2" layer="1"/>
-<wire x1="55.2481" y1="50.01440625" x2="55.51250625" y2="49.75" width="0.2" layer="1"/>
 <wire x1="55.51250625" y1="49.75" x2="56.238" y2="49.75" width="0.2" layer="1"/>
 <wire x1="20.35" y1="31.7" x2="20.35" y2="29.6" width="0.2" layer="1"/>
+<wire x1="55.51250625" y1="49.75" x2="53.25" y2="52.01250625" width="0.2" layer="1"/>
+<wire x1="53.25" y1="52.01250625" x2="53.25" y2="53.238" width="0.2" layer="1"/>
+<wire x1="53.01440625" y1="52.2481" x2="53.25" y2="52.01250625" width="0.2" layer="1"/>
+<wire x1="47.01440625" y1="52.2481" x2="53.01440625" y2="52.2481" width="0.2" layer="1"/>
+<wire x1="62.5" y1="44.75" x2="63.625" y2="45.875" width="0.2" layer="1"/>
+<wire x1="63.625" y1="45.875" x2="63.625" y2="46.65" width="0.2" layer="1"/>
 <wire x1="42" y1="55.75" x2="44.5" y2="55.15" width="0" layer="19" extent="1-1"/>
 <wire x1="58.15" y1="41.18" x2="62.5" y2="44.75" width="0" layer="19" extent="1-1"/>
@@
 <wire x1="42.23650625" y1="50.25" x2="40.58650625" y2="48.6" width="0.2" layer="1"/>
 <wire x1="40.58650625" y1="48.6" x2="39.701625" y2="48.6" width="0.2" layer="1"/>
-<wire x1="45.65318125" y1="50.15" x2="46.5519" y2="49.25128125" width="0.2" layer="1"/>
 <wire x1="46.5519" y1="49.25128125" x2="46.5519" y2="43.18303125" width="0.2" layer="1"/>
-<wire x1="44.762" y1="50.25" x2="44.862" y2="50.15" width="0.2" layer="1"/>
-<wire x1="44.862" y1="50.15" x2="45.65318125" y2="50.15" width="0.2" layer="1"/>
 <wire x1="46.5519" y1="43.18303125" x2="44.562" y2="41.19313125" width="0.2" layer="1"/>
 <via x="42" y="31.27321875" extent="1-16" drill="0.35"/>
@@
 <wire x1="43.6944" y1="27.9856" x2="42.68" y2="29" width="0.2" layer="16"/>
 <wire x1="45.2444" y1="27.9856" x2="43.6944" y2="27.9856" width="0.2" layer="16"/>
+<wire x1="44.762" y1="50.25" x2="45.55318125" y2="50.25" width="0.2" layer="1"/>
+<wire x1="45.55318125" y1="50.25" x2="46.5519" y2="49.25128125" width="0.2" layer="1"/>
 </signal>
 <signal name="MOSI">
@@
 <contactref element="JP1" pad="18"/>
 <via x="42.445903125" y="48.445903125" extent="1-16" drill="0.35"/>
-<wire x1="44.762" y1="48.75" x2="44.6494" y2="48.6374" width="0.2" layer="1"/>
-<wire x1="44.6494" y1="48.6374" x2="43.92390625" y2="48.6374" width="0.2" layer="1"/>
-<wire x1="43.732409375" y1="48.445903125" x2="42.445903125" y2="48.445903125" width="0.2" layer="1"/>
-<wire x1="43.92390625" y1="48.6374" x2="43.732409375" y2="48.445903125" width="0.2" layer="1"/>
 <wire x1="41.0306" y1="50.10989375" x2="40.42689375" y2="50.7136" width="0.2" layer="16"/>
 <wire x1="42.445903125" y1="48.445903125" x2="41.0306" y2="49.86120625" width="0.2" layer="16"/>
@@
 <wire x1="13.42981875" y1="47.9044" x2="12.41541875" y2="46.89" width="0.2" layer="16"/>
 <wire x1="36.74656875" y1="48.3156" x2="15.2156" y2="48.3156" width="0.2" layer="16"/>
+<wire x1="44.762" y1="48.75" x2="43.64180625" y2="48.75" width="0.2" layer="1"/>
+<wire x1="43.64180625" y1="48.75" x2="43.337709375" y2="48.445903125" width="0.2" layer="1"/>
+<wire x1="43.337709375" y1="48.445903125" x2="42.445903125" y2="48.445903125" width="0.2" layer="1"/>
 </signal>
 <signal name="SDA">
@@
 <wire x1="40.42761875" y1="32.07238125" x2="40.42761875" y2="30.07238125" width="0.2" layer="1"/>
 <via x="40.42761875" y="30.07238125" extent="1-16" drill="0.35"/>
-<wire x1="45.60009375" y1="47.6374" x2="45.7519" y2="47.48559375" width="0.2" layer="1"/>
-<wire x1="44.762" y1="47.75" x2="44.8746" y2="47.6374" width="0.2" layer="1"/>
-<wire x1="44.8746" y1="47.6374" x2="45.60009375" y2="47.6374" width="0.2" layer="1"/>
 <wire x1="43.762" y1="41.52450625" x2="43.762" y2="35.4067625" width="0.2" layer="1"/>
 <wire x1="45.7519" y1="47.48559375" x2="45.7519" y2="43.51440625" width="0.2" layer="1"/>
@@
 <wire x1="40.42761875" y1="30.07238125" x2="40.42761875" y2="29.8178" width="0.2" layer="16"/>
 <wire x1="40.42761875" y1="29.8178" x2="44.1756" y2="26.06981875" width="0.2" layer="16"/>
+<wire x1="44.762" y1="47.75" x2="45.48749375" y2="47.75" width="0.2" layer="1"/>
+<wire x1="45.48749375" y1="47.75" x2="45.7519" y2="47.48559375" width="0.2" layer="1"/>
 <wire x1="44.542759375" y1="23.9572375" x2="45.8469875" y2="22.55236875" width="0" layer="19" extent="1-1"/>
 </signal>
@@
 <wire x1="58.15" y1="47.5" x2="57.4" y2="46.75" width="0.2" layer="1"/>
 <wire x1="57.4" y1="46.75" x2="56.238" y2="46.75" width="0.2" layer="1"/>
-<wire x1="55.39990625" y1="46.6374" x2="55.2481" y2="46.48559375" width="0.2" layer="1"/>
 <wire x1="58.75455" y1="41.9824" x2="58.9024" y2="41.83455" width="0.2" layer="1"/>
 <wire x1="58.9024" y1="41.83455" x2="58.9024" y2="40.52545" width="0.2" layer="1"/>
-<wire x1="56.238" y1="46.75" x2="56.1254" y2="46.6374" width="0.2" layer="1"/>
-<wire x1="56.1254" y1="46.6374" x2="55.39990625" y2="46.6374" width="0.2" layer="1"/>
 <wire x1="55.2481" y1="46.48559375" x2="55.2481" y2="42.67495" width="0.2" layer="1"/>
 <wire x1="58.9024" y1="40.52545" x2="58" y2="39.62305" width="0.2" layer="1"/>
@@
 <wire x1="21.1024" y1="32.35455" x2="21.1024" y2="31.0386" width="0.2" layer="1"/>
 <wire x1="20.95455" y1="32.5024" x2="18.04545" y2="32.5024" width="0.2" layer="1"/>
+<wire x1="56.238" y1="46.75" x2="55.51250625" y2="46.75" width="0.2" layer="1"/>
+<wire x1="55.51250625" y1="46.75" x2="55.2481" y2="46.48559375" width="0.2" layer="1"/>
 </signal>
 <signal name="FEEDBACK_DA">

Commit message: Все платы проверены и вроеде бы как готовы к изготовлению!
Parts:
- removed LED1, LED2: (no value), led:CHIPLED_0603
- removed U$10, U$11, U$13, U$15, U$18, U$19, U$4, U$9: MOSFET-N, NEON-BLADE-2023:SOT23-3
- added 3V3, 5V: (no value), NEON-BLADE-2023:VIAS-CONNECT
- added PC13, PWR: (no value), led:CHIPLED_0603
- added R36, R37: 4k7, rcl:R0603
- added SI2301, SI2301.2, SI2301.3, SI2301.4, SI2301.5, SI2301.6, SI2301.7, SI2301.8: MOSFET-N, NEON-BLADE-2023:SOT23-3
- C9: value 100nf -> 100nF
- R17: value 191k -> 191k/2k
- R32: value 10k -> 3k9
- moved JP3 50.8 mm to (3.40, 62.1)
- moved R32 31.7 mm to (37.0, 64.0), turned to 90 degrees
- moved JP2 27.4 mm to (11.0, 12.0), flipped to the top, turned to 180 degrees
- moved R3 24.9 mm to (59.1, 41.2), turned to 0 degrees
- moved C2 23.6 mm to (41.1, 55.3), turned to 90 degrees
- moved R25 10.9 mm to (21.9, 50.7)
- moved R28 7.53 mm to (31.7, 51.3), turned to 90 degrees
- moved R19 6.71 mm to (3.90, 52.3)
- moved R14 6.23 mm to (11.6, 17.3), turned to 90 degrees
- moved R16 6.23 mm to (13.7, 17.3), turned to 270 degrees
- moved R12 6.20 mm to (12.2, 23.2)
- moved R6 5.83 mm to (41.5, 42.0), turned to 180 degrees
- moved R22 5.51 mm to (13.7, 53.0), turned to 90 degrees
- moved R31 5.47 mm to (43.3, 56.2), turned to 270 degrees
- moved R21 4.72 mm to (4.40, 58.2), turned to 270 degrees
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- renumbered IC1 to STM32F401, U$1 to LIS3MDL, U$14 to PHOTORES, U$2 to LSM6DS3, U$3 to BUZZER, U$5 to MICROSD, U$6 to DC-DC_5V, U$7 to DC-DC_3V3
Connections:
- new net N$13: 3V3.2, 5V.1, R17.1
- net 3V3: now also 3V3.1, PC13.A, PWR.A, R36.2, R37.2; no longer LED1.A, LED2.A
- net 5V: now also 5V.2; no longer R17.1
- net BOTTON_DA_DOWN: now also SI2301.7.3; no longer U$4.3
- net BOTTON_DA_UP: now also SI2301.8.3; no longer U$9.3
- net BOTTON_PAR_DOWN: now also SI2301.4.3; no longer U$10.3
- net BOTTON_PAR_UP: now also SI2301.5.3; no longer U$11.3
- net BOTTON_SKIRT_CLOSE: now also SI2301.2.3; no longer U$13.3
- net BOTTON_SKIRT_OPEN: now also SI2301.3.3; no longer U$15.3
- net CE_NRF: now also STM32F401.9
- net CS_NRF: now also STM32F401.8
- net ESP_EN: now also STM32F401.33
- net FEEDBACK_DA: now also STM32F401.50, U$8.P$4; no longer U$8.P$3
- net FEEDBACK_SKIRT: now also STM32F401.24
- net GND: now also SI2301.2, SI2301.2.2, SI2301.3.2, SI2301.4.2, SI2301.5.2, SI2301.6.2, SI2301.7.2, SI2301.8.2, U$8.P$3; no longer U$10.2, U$11.2, U$13.2, U$15.2, U$18.2, U$19.2, U$4.2, U$8.P$4, U$9.2
- net GND_ESP: now also SI2301.6.3; no longer U$19.3
- net KO: now also STM32F401.22
- net MOTOR_DA_DOWN: now also STM32F401.44
- net MOTOR_DA_UP: now also STM32F401.45
- net MOTOR_PAR_DOWN: now also STM32F401.26
- net MOTOR_PAR_UP: now also STM32F401.25
- net MOTOR_SKIRT_CLOSE: now also STM32F401.28
- net MOTOR_SKIRT_OPEN: now also STM32F401.27
- net N$1: now also SI2301.1; no longer U$18.1
- net N$11: now also SI2301.5.1; no longer U$11.1
- net N$14: now also SI2301.2.1; no longer U$13.1
- net N$17: now also SI2301.3.1; no longer U$15.1
- net N$2: now also SI2301.7.1; no longer U$4.1
- net N$20: now also SI2301.3; no longer U$18.3
- net N$3: now also SI2301.4.1; no longer U$10.1
- net N$36: now also PWR.C; no longer LED1.C
- net N$37: now also PC13.C; no longer LED2.C
- net N$4: now also SI2301.6.1; no longer U$19.1
- net N$8: now also SI2301.8.1; no longer U$9.1
- net NRF_IRQ: now also STM32F401.11
- net SCL: now also R37.1
- net SDA: now also R36.1
- net STATE: now also STM32F401.41
- net USIL_ON: now also STM32F401.62
Routing:
- net GND: track 102.6 -> 351.9 mm, vias 2 -> 20
- net 5V: track 41.7 -> 211.9 mm, vias 5 -> 3
- net 3V3: track 82.2 -> 192.0 mm, vias 0 -> 6
- net FEEDBACK_SKIRT: track 5.16 -> 89.4 mm, vias 0 -> 3
- net MOTOR_PAR_UP: track 0.00 -> 75.2 mm, vias 0 -> 6
- net MOTOR_DA_DOWN: track 0.00 -> 70.1 mm, vias 0 -> 4
- net CS_NRF: track 0.00 -> 66.8 mm, vias 0 -> 1
- net CE_NRF: track 0.00 -> 65.1 mm, vias 0 -> 1
- net N$9: track 81.6 -> 17.8 mm
- net N$5: track 72.2 -> 11.3 mm
- net USIL_ON: track 0.00 -> 58.0 mm, vias 0 -> 3
- net MOTOR_PAR_DOWN: track 0.00 -> 55.9 mm, vias 0 -> 4
- net MOTOR_DA_UP: track 0.00 -> 54.6 mm, vias 0 -> 2
- net KO: track 0.00 -> 54.1 mm, vias 0 -> 4
- net STATE: track 0.00 -> 48.6 mm, vias 0 -> 2
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- added copper zone on layer 1, net GND
- added copper zone on layer 16, net GND
Other:
- board size 68.5 x 75.2 mm -> 68 x 75.2 mm
- board text added: "3V3"
- board text added: "5V"
- board text added: "BT_PAR_DW"
- board text added: "BT_PAR_UP"
- board text added: "BT_SK_CL"
- board text added: "BT_SK_OP"
- board text added: "CE_NRF"
- board text added: "CS_LIS"
- board text added: "CS_NRF"
- board text added: "DBG_RX"
- board text added: "DBG_TX"
- board text added: "FB SK"
- board text added: "FB_DA"
- board text added: "FFC to ESP32-CAM"
- board text added: "G RX"
- board text added: "G TX"
- board text added: "GND"
- board text added: "KO"
- board text added: "MISO"
- board text added: "MOSI"
- board text added: "MOT DA"
- board text added: "MOT PAR"
- board text added: "N IRQ"
- board text added: "PH3V3"
- board text added: "PH5V"
- board text added: "PSK CL"
- board text added: "PSK OP"
- board text added: "SCK"
- board text added: "SCL"
- board text added: "SDA"
- board text added: "STATE"
- board text added: "USIL_ON"
- board text added: "|3V3"
- board text added: "|BT_DA_DW"
- board text added: "|BT_DA_UP"
- board text added: "|FB_SKIRT"
- board text added: "|GND"
- board text added: "|NRST"
- board text added: "|SVC"
- board text added: "|SVD"
- board text added: "|V_BAT"
