File: schematics/board/MA_board_1.sch (EAGLE design)
At the start: 69 parts, among them IC1 STM32F401RCT6

Commit message: новая версия первой платы нижнего модуля
Parts:
- removed R1: 10k, rcl:R-EU_R0603
- added C10: 10nF, rcl:C-EUC0603
- added C11: 4.7uf, rcl:C-EUC0603
- added C12, C13: 100nF, rcl:C-EUC0603
- added C8: 1nF, rcl:C-EUC0603
- added C9: 100nf, rcl:C-EUC0603
- added Q24: Q24, CanCubeSat:Q24
- R17: value 100R -> 191k
- U$1: value LIS3MDL_CJMCU -> LIS3MDL-CJMCUБез_отв._зеркальный; device NEON-BLADE-2023:LIS3MDL_CJMCU -> NEON-BLADE-2023:LIS3MDL-CJMCUБез_отв._зеркальный
- U$2: value LSM6DS3-GY -> LSM6DS3-GY-NB2023; device NEON-BLADE-2023:LSM6DS3-GY -> NEON-BLADE-2023:LSM6DS3-GY-NB2023
Connections:
- net BUTTON_DA_UP renamed FEEDBACK_DA
- net DA_DOWN_ON renamed BOTTON_DA_DOWN
- net DA_UP_ON renamed BOTTON_DA_UP
- net PAR_DOWN_ON renamed BOTTON_PAR_DOWN
- net PAR_UP_ON renamed BOTTON_PAR_UP
- net SKIRT_CLOSE_ON renamed BOTTON_SKIRT_CLOSE
- net SKIRT_OPEN_ON renamed BOTTON_SKIRT_OPEN
- removed net BUTTON_DA_DOWN: JP1.2, U$8.4
- removed net BUTTON_SKIRT_CLOSE: JP1.3, JP7.6
- removed net BUTTON_SKIRT_OPEN: JP1.5, JP7.5
- removed net N$35: IC1.NRST, R1.2
- new net FEEDBACK_SKIRT: C12.2, JP1.3, JP7.6
- new net FEEDBACK_SKIRT1: C13.2
- new net N$10: C8.2, Q24.OUTPUT
- new net N$12: C11.1, IC1.VCAP_1
- new net NRST: C9.2, IC1.NRST, JP1.5
- new net TCXO: C8.1, IC1.PH0-OSC_IN
- net 3V3: now also C10.2, Q24.VCC; no longer R1.1
- net GND: now also C10.1, C11.2, C12.1, C13.1, C9.1, Q24.GND
Other:
- moved on the sheet: JP2, R11, R12, R13, R14, R15, R16, U$16, U$4, U$9

Commit message: немного продвинул работу над платой (Прмгите)
Parts:
- removed C12, C13: 100nF, rcl:C-EUC0603
- added R1, R35: 10k, rcl:R-EU_R0603
Connections:
- removed net FEEDBACK_SKIRT1: C13.2
- new net NRF_IRQ: JP7.5
- net 3V3: now also R1.2, R35.1
- net CE_NRF: no longer IC1.PC13
- net CS_NRF: no longer IC1.PC14-_OSC32_IN
- net FEEDBACK_DA: now also R35.2
- net FEEDBACK_SKIRT: now also R1.1; no longer C12.2
- net GND: now also U$8.4; no longer C12.1, C13.1
- net LED: now also IC1.PC13
- net MOSI: now also JP6.3; no longer JP6.1
- net SCK: now also JP6.1; no longer JP6.3
Changed lines of the file:
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@@
 <part name="C9" library="rcl" library_urn="urn:adsk.eagle:library:334" deviceset="C-EU" device="C0603" package3d_urn="urn:adsk.eagle:package:23616/2" value="100nf"/>
 <part name="C11" library="rcl" library_urn="urn:adsk.eagle:library:334" deviceset="C-EU" device="C0603" package3d_urn="urn:adsk.eagle:package:23616/2" value="4.7uf"/>
-<part name="C12" library="rcl" library_urn="urn:adsk.eagle:library:334" deviceset="C-EU" device="C0603" package3d_urn="urn:adsk.eagle:package:23616/2" value="100nF"/>
-<part name="C13" library="rcl" library_urn="urn:adsk.eagle:library:334" deviceset="C-EU" device="C0603" package3d_urn="urn:adsk.eagle:package:23616/2" value="100nF"/>
+<part name="R1" library="rcl" library_urn="urn:adsk.eagle:library:334" deviceset="R-EU_" device="R0603" package3d_urn="urn:adsk.eagle:package:23555/3" value="10k"/>
+<part name="R35" library="rcl" library_urn="urn:adsk.eagle:library:334" deviceset="R-EU_" device="R0603" package3d_urn="urn:adsk.eagle:package:23555/3" value="10k"/>
 </parts>
 <sheets>
@@
 <attribute name="VALUE" x="90.424" y="-2.159" size="1.778" layer="96"/>
 </instance>
-<instance part="C12" gate="G$1" x="180.34" y="86.36" smashed="yes" rot="R90">
-<attribute name="NAME" x="178.816" y="85.979" size="1.778" layer="95" rot="R180"/>
-<attribute name="VALUE" x="178.816" y="88.519" size="1.778" layer="96" rot="R180"/>
-</instance>
-<instance part="C13" gate="G$1" x="241.3" y="86.36" smashed="yes" rot="MR90">
-<attribute name="NAME" x="242.824" y="85.979" size="1.778" layer="95" rot="MR180"/>
-<attribute name="VALUE" x="242.824" y="88.519" size="1.778" layer="96" rot="MR180"/>
+<instance part="R1" gate="G$1" x="180.34" y="86.36" smashed="yes" rot="R180">
+<attribute name="NAME" x="181.61" y="87.4014" size="1.778" layer="95" rot="R180"/>
+<attribute name="VALUE" x="176.53" y="84.582" size="1.778" layer="96" rot="R180"/>
+</instance>
+<instance part="R35" gate="G$1" x="238.76" y="91.44" smashed="yes" rot="R180">
+<attribute name="NAME" x="237.49" y="95.0214" size="1.778" layer="95" rot="R180"/>
+<attribute name="VALUE" x="242.57" y="94.742" size="1.778" layer="96" rot="R180"/>
 </instance>
 </instances>
@@
 <pinref part="C10" gate="G$1" pin="2"/>
 </segment>
+<segment>
+<pinref part="R1" gate="G$1" pin="2"/>
+<wire x1="175.26" y1="86.36" x2="170.18" y2="86.36" width="0.1524" layer="91"/>
+<label x="170.18" y="86.36" size="1.778" layer="95"/>
+</segment>
+<segment>
+<pinref part="R35" gate="G$1" pin="1"/>
+<wire x1="243.84" y1="91.44" x2="248.92" y2="91.44" width="0.1524" layer="91"/>
+<label x="243.84" y="91.44" size="1.778" layer="95"/>
+</segment>
 </net>
 <net name="GND" class="0">
@@
 </segment>
 <segment>
-<pinref part="C12" gate="G$1" pin="1"/>
-<wire x1="177.8" y1="86.36" x2="165.1" y2="86.36" width="0.1524" layer="91"/>
-<label x="172.72" y="86.36" size="1.778" layer="95" rot="R180"/>
-</segment>
-<segment>
-<pinref part="C13" gate="G$1" pin="1"/>
-<wire x1="243.84" y1="86.36" x2="251.46" y2="86.36" width="0.1524" layer="91"/>
-<label x="248.92" y="86.36" size="1.778" layer="95" rot="MR180"/>
+<pinref part="U$8" gate="G$1" pin="4"/>
+<wire x1="200.66" y1="50.8" x2="175.26" y2="50.8" width="0.1524" layer="91"/>
+<label x="175.26" y="50.8" size="1.778" layer="95"/>
 </segment>
 </net>
@@
 <wire x1="139.7" y1="12.7" x2="134.62" y2="12.7" width="0.1524" layer="91"/>
 <label x="135.128" y="13.462" size="1.778" layer="95"/>
+</segment>
+<segment>
+<pinref part="IC1" gate="G$1" pin="PC13"/>
+<wire x1="48.26" y1="76.2" x2="30.48" y2="76.2" width="0.1524" layer="91"/>
+<label x="30.48" y="76.2" size="1.778" layer="95"/>
 </segment>
 </net>
@@
 </segment>
 <segment>
-<pinref part="JP6" gate="A" pin="3"/>
-<wire x1="160.02" y1="76.2" x2="149.86" y2="76.2" width="0.1524" layer="91"/>
-<label x="147.32" y="76.2" size="1.778" layer="95"/>
-</segment>
-<segment>
 <pinref part="U$2" gate="G$1" pin="SCL"/>
 <wire x1="139.7" y1="-35.56" x2="154.94" y2="-35.56" width="0.1524" layer="91"/>
@@
 <label x="83.82" y="-27.94" size="1.778" layer="95"/>
 </segment>
+<segment>
+<pinref part="JP6" gate="A" pin="1"/>
+<wire x1="160.02" y1="71.12" x2="149.86" y2="71.12" width="0.1524" layer="91"/>
+<label x="149.86" y="71.12" size="1.778" layer="95"/>
+</segment>
 </net>
 <net name="MISO" class="0">
@@
 <pinref part="JP6" gate="A" pin="2"/>
 <wire x1="160.02" y1="73.66" x2="149.86" y2="73.66" width="0.1524" layer="91"/>
-<label x="147.32" y="73.66" size="1.778" layer="95"/>
+<label x="149.86" y="73.66" size="1.778" layer="95"/>
 </segment>
 <segment>
@@
 </segment>
 <segment>
-<pinref part="JP6" gate="A" pin="1"/>
-<wire x1="160.02" y1="71.12" x2="149.86" y2="71.12" width="0.1524" layer="91"/>
-<label x="147.32" y="71.12" size="1.778" layer="95"/>
-</segment>
-<segment>
 <pinref part="U$1" gate="G$1" pin="SDA(MOSI)"/>
 <wire x1="78.74" y1="-33.02" x2="93.98" y2="-33.02" width="0.1524" layer="91"/>
@@
 <label x="144.78" y="-40.64" size="1.778" layer="95"/>
 </segment>
+<segment>
+<pinref part="JP6" gate="A" pin="3"/>
+<wire x1="160.02" y1="76.2" x2="149.86" y2="76.2" width="0.1524" layer="91"/>
+<label x="149.86" y="76.2" size="1.778" layer="95"/>
+</segment>
 </net>
 <net name="CS_NRF" class="0">
@@
 <label x="147.32" y="78.74" size="1.778" layer="95"/>
 </segment>
-<segment>
-<pinref part="IC1" gate="G$1" pin="PC14-_OSC32_IN"/>
-<wire x1="48.26" y1="73.66" x2="30.48" y2="73.66" width="0.1524" layer="91"/>
-<label x="30.48" y="73.66" size="1.778" layer="95"/>
-</segment>
 </net>
 <net name="CE_NRF" class="0">
@@
 <wire x1="160.02" y1="81.28" x2="149.86" y2="81.28" width="0.1524" layer="91"/>
 <label x="147.32" y="81.28" size="1.778" layer="95"/>
-</segment>
-<segment>
-<pinref part="IC1" gate="G$1" pin="PC13"/>
-<wire x1="48.26" y1="76.2" x2="30.48" y2="76.2" width="0.1524" layer="91"/>
-<label x="30.48" y="76.2" size="1.778" layer="95"/>
 </segment>
 </net>
@@
 <pinref part="JP1" gate="A" pin="3"/>
 <label x="175.26" y="88.9" size="1.778" layer="95"/>
-<wire x1="200.66" y1="88.9" x2="187.96" y2="88.9" width="0.1524" layer="91"/>
-<wire x1="187.96" y1="88.9" x2="187.96" y2="86.36" width="0.1524" layer="91"/>
-<junction x="187.96" y="88.9"/>
-<wire x1="187.96" y1="86.36" x2="185.42" y2="86.36" width="0.1524" layer="91"/>
-<pinref part="C12" gate="G$1" pin="2"/>
-<wire x1="187.96" y1="88.9" x2="177.8" y2="88.9" width="0.1524" layer="91"/>
+<wire x1="200.66" y1="88.9" x2="185.42" y2="88.9" width="0.1524" layer="91"/>
+<pinref part="R1" gate="G$1" pin="1"/>
+<wire x1="185.42" y1="88.9" x2="177.8" y2="88.9" width="0.1524" layer="91"/>
+<wire x1="185.42" y1="86.36" x2="185.42" y2="88.9" width="0.1524" layer="91"/>
+<junction x="185.42" y="88.9"/>
 </segment>
 <segment>
@@
 <pinref part="JP1" gate="A" pin="4"/>
 <label x="213.36" y="88.9" size="1.778" layer="95"/>
-<wire x1="208.28" y1="88.9" x2="238.76" y2="88.9" width="0.1524" layer="91"/>
+<wire x1="208.28" y1="88.9" x2="233.68" y2="88.9" width="0.1524" layer="91"/>
+<pinref part="R35" gate="G$1" pin="2"/>
+<wire x1="233.68" y1="88.9" x2="233.68" y2="91.44" width="0.1524" layer="91"/>
+<junction x="233.68" y="88.9"/>
+<wire x1="233.68" y1="88.9" x2="243.84" y2="88.9" width="0.1524" layer="91"/>
 </segment>
 <segment>
@@
 <wire x1="88.9" y1="22.86" x2="88.9" y2="5.08" width="0.1524" layer="91"/>
 <pinref part="C11" gate="G$1" pin="1"/>
-</segment>
-</net>
-<net name="FEEDBACK_SKIRT1" class="0">
-<segment>
-<wire x1="233.68" y1="88.9" x2="233.68" y2="86.36" width="0.1524" layer="91"/>
-<wire x1="233.68" y1="86.36" x2="236.22" y2="86.36" width="0.1524" layer="91"/>
-<pinref part="C13" gate="G$1" pin="2"/>
 </segment>
 </net>
@@
 </segment>
 </net>
+<net name="NRF_IRQ" class="0">
+<segment>
+<pinref part="JP7" gate="A" pin="5"/>
+<wire x1="160.02" y1="55.88" x2="142.24" y2="55.88" width="0.1524" layer="91"/>
+<label x="142.24" y="55.88" size="1.778" layer="95"/>
+</segment>
+</net>

Commit message: Все платы проверены и вроеде бы как готовы к изготовлению!
Parts:
- added 3V3, 5V: (no value), NEON-BLADE-2023:VIAS-CONNECT
- added R36, R37: 4k7, rcl:R-EU_R0603
- C9: value 100nf -> 100nF
- R17: value 191k -> 191k/2k
- R32: value 10k -> 3k9
- renumbered IC1 to STM32F401, LED1 to PWR, LED2 to PC13, U$1 to LIS3MDL, U$10 to SI2301.4, U$11 to SI2301.5, U$13 to SI2301.2, U$14 to PHOTORES, U$15 to SI2301.3, U$18 to SI2301, U$19 to SI2301.6, U$2 to LSM6DS3, U$3 to BUZZER, U$4 to SI2301.7, U$5 to MICROSD, U$6 to DC-DC_5V, U$7 to DC-DC_3V3, U$9 to SI2301.8
Connections:
- new net N$13: 3V3.2, 5V.1, R17.1
- net 3V3: now also 3V3.1, R36.2, R37.2
- net 5V: now also 5V.2; no longer R17.1
- net CE_NRF: now also STM32F401.PC1
- net CS_NRF: now also STM32F401.PC0
- net ESP_EN: now also STM32F401.PB12
- net FEEDBACK_DA: now also STM32F401.PA15, U$8.4; no longer U$8.3
- net FEEDBACK_SKIRT: now also STM32F401.PC4
- net GND: now also U$8.3; no longer U$8.4
- net KO: now also STM32F401.PA6
- net MOTOR_DA_DOWN: now also STM32F401.PA11
- net MOTOR_DA_UP: now also STM32F401.PA12
- net MOTOR_PAR_DOWN: now also STM32F401.PB0
- net MOTOR_PAR_UP: now also STM32F401.PC5
- net MOTOR_SKIRT_CLOSE: now also STM32F401.PB2
- net MOTOR_SKIRT_OPEN: now also STM32F401.PB1
- net NRF_IRQ: now also STM32F401.PC3
- net SCL: now also R37.1
- net SDA: now also R36.1
- net STATE: now also STM32F401.PA8
- net USIL_ON: now also STM32F401.PB9
Other:
- moved on the sheet: C9, R1, R35

Commit message: Еще раз проверил все платы и подготовил для производства в Резоните
Parts:
- JP2, JP3, JP4: value (none) -> JST-2-K-S; device pinhead:PINHD-1X2 -> NEON-BLADE-2023:JST-2-K-S
- JP6, JP7: device pinhead:PINHD-1X8 -> NEON-BLADE-2023:PINHD-1X8-SHORT-PAD
Connections:
- net N$5: now also JP4.2; no longer JP4.1
- net N$9: now also JP4.1; no longer JP4.2
Other:
- moved on the sheet: JP2, JP3, JP4
