File: schematics/board/MA_board_2.brd (EAGLE design)
At the start: 68 x 55 mm, 23 parts, among them J1 MCX-J-P-H-ST-TH1, J2 U.FL-R-SMT-1_10_

Commit message: Проверил платы. Исправил некоторые ошибки
Parts:
- removed JP3, JP5, JP6: (no value), pinhead:1X02
- added BATTERY, GENERATOR, MOTOR: (no value), pinhead:1X02
- added C3: 100nF, rcl:C0603
- added D1: DIODE-MBR, NEON-BLADE-2023:SOD123
- C2: value 100NF -> 100nF
- R3: device rcl:R2012 -> rcl:R2512
- moved R2 117.8 mm to (56.9, 27.9), turned to 270 degrees
- moved U$1 117.5 mm to (57.3, 22.5), turned to 270 degrees
- moved R3 113.9 mm to (58.0, 31.5), turned to 180 degrees
- moved R1 112.5 mm to (59.1, 27.9), turned to 270 degrees
- moved C2 90.9 mm to (58.0, 25.3), turned to 180 degrees
- moved LED1 40.4 mm to (-23.6, 18.7)
- moved LED2 40.4 mm to (-23.6, 8.53)
- moved R4 40.4 mm to (-24.9, 14.9)
- moved R5 40.4 mm to (-24.9, 4.72)
- moved U$2 8.75 mm to (-23.0, 55.2)
- flipped JP1 to the bottom, turned to 180 degrees
- flipped JP2 to the bottom, turned to 0 degrees
- renumbered JP4 to B_CLOSE, JP7 to B_OPEN
Connections:
- new net N$8: D1.A, R2.1, R3.2
- net 3V3: now also C3.2; no longer U$4.P$8, U$4.P$9
- net GND: now also BATTERY.2, C3.1, GENERATOR.2, J2.1; no longer JP5.2, JP6.2
- net LED1: now also U$4.P$8
- net LED2: now also U$4.P$9
- net N$4: now also GENERATOR.1; no longer JP6.1
- net N$6: now also BATTERY.1, D1.C; no longer JP5.1, R2.1, R3.2
- net POWER_SKIRT_CLOSE: now also MOTOR.1; no longer JP3.1
- net POWER_SKIRT_OPEN: now also MOTOR.2; no longer JP3.2

Commit message: Я Данижок, и я тоже сделал плату. А куратор за всех коммитит и выключает компьютеры((
Parts:
- removed U$2: REF3033, NEON-BLADE-2023:SOT23-3
- added REF3033: REF3033, NEON-BLADE-2023:SOT23-3
- moved C1 55.5 mm to (35.6, 48.5), turned to 90 degrees
- moved R4 40.5 mm to (13.6, 2.30), turned to 270 degrees
- moved LED1 39.5 mm to (13.6, 5.50), turned to 270 degrees
- moved R5 36.5 mm to (11.5, 2.30), turned to 270 degrees
- moved LED2 35.3 mm to (11.5, 5.50), turned to 270 degrees
- moved C2 0.50 mm to (57.5, 25.3)
- moved R1 0.50 mm to (58.6, 27.9)
- moved R2 0.50 mm to (56.4, 27.9)
- moved R3 0.50 mm to (57.5, 31.5)
- turned C3 to 90 degrees
- renumbered B_CLOSE to B_CL, B_OPEN to B_OP, U$1 to INA219, U$4 to AMP
Connections:
- net 3V3: now also REF3033.2; no longer U$2.2
- net 5V: now also REF3033.1; no longer U$2.1
- net GND: now also REF3033.3; no longer U$2.3
Routing:
- net GND: track 0.00 -> 284.0 mm, vias 0 -> 8
- net 3V3: track 0.00 -> 117.8 mm, vias 0 -> 3
- net 5V: track 0.00 -> 62.3 mm
- net USIL_ON: track 0.00 -> 52.2 mm
- net NRF_IRQ: track 0.00 -> 45.2 mm, vias 0 -> 2
- net SDA: track 0.00 -> 42.0 mm
- net SCL: track 0.00 -> 40.1 mm, vias 0 -> 1
- net N$4: track 0.00 -> 32.1 mm
- net CE_NRF: track 0.00 -> 31.6 mm, vias 0 -> 1
- net CS_NRF: track 0.00 -> 27.3 mm, vias 0 -> 1
- net FEEDBACK_SKIRT: track 0.00 -> 26.2 mm, vias 0 -> 1
- net N$8: track 0.00 -> 23.2 mm
- net MOSI: track 0.00 -> 22.5 mm, vias 0 -> 1
- net SCK: track 0.00 -> 20.5 mm
- net MISO: track 0.00 -> 20.5 mm
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- added copper zone on layer 1, net GND
- added copper zone on layer 16, net GND
Other:
- board text added: "5V"
- board text added: "ANT"
- board text added: "CE_NRF"
- board text added: "CS_NRF"
- board text added: "GND"
- board text added: "MISO"
- board text added: "MOSI"
- board text added: "SCK"
- board text added: "USIL_ON"
- board text added: "nRF24"

Commit message: Все платы проверены и вроеде бы как готовы к изготовлению!
Parts:
- removed B_CL, B_OP: (no value), pinhead:1X02
- added BUTTON-OP, BUTTONS: JST-2-K-S, NEON-BLADE-2023:B2B-PH-K-S
- added C4: 220uF, NEON-BLADE-2023:ECAP220-CMD
- added C6: 100nF, rcl:C0603
- BATTERY, GENERATOR, MOTOR: value (none) -> JST-2-K-S; device pinhead:1X02 -> NEON-BLADE-2023:B2B-PH-K-S
- D1: value DIODE-MBR -> D-MBR
- JP1, JP2: device pinhead:1X08 -> NEON-BLADE-2023:1X08
- moved INA219 26.1 mm to (31.2, 23.5)
- moved C3 25.9 mm to (28.7, 23.5)
- moved C2 25.6 mm to (31.9, 26.3)
- moved R1 25.6 mm to (33.0, 28.9)
- moved R3 25.6 mm to (31.9, 32.5)
- moved R2 25.6 mm to (30.8, 28.9)
- moved GENERATOR 22.7 mm to (29.5, 48.0)
- moved MOTOR 21.0 mm to (38.9, 7.50)
- moved D1 15.9 mm to (34.2, 38.4), turned to 180 degrees
- moved C1 15.9 mm to (51.4, 49.5), turned to 270 degrees
- moved U$5 10.5 mm to (50.0, 27.5)
- moved REF3033 9.98 mm to (48.5, 49.3), turned to 180 degrees
- moved BATTERY 8.14 mm to (37.5, 48.0)
- moved J2 1.00 mm to (9.00, 50.3)
- moved AMP 0.50 mm to (13.5, 28.0)
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- renumbered U$3 to NRF24L01P
Connections:
- net 5V: now also C4.P$1, C6.2
- net FEEDBACK_SKIRT: now also BUTTON-OP.2, BUTTONS.1; no longer B_CL.1, B_OP.1
- net GND: now also BUTTON-OP.1, BUTTONS.2, C4.P$2, C6.1; no longer B_CL.2, B_OP.2
Routing:
- net 3V3: track 117.8 -> 78.1 mm
- net POWER_SKIRT_CLOSE: track 4.05 -> 27.0 mm
- net 5V: track 62.3 -> 84.4 mm
- net SDA: track 42.0 -> 22.1 mm
- net MISO: track 20.5 -> 40.1 mm
- net MOSI: track 22.5 -> 40.7 mm, vias 1 -> 0
- net SCL: track 40.1 -> 22.4 mm, vias 1 -> 0
- net SCK: track 20.5 -> 38.0 mm, vias 0 -> 1
- net POWER_SKIRT_OPEN: track 4.05 -> 21.0 mm
- net NRF_IRQ: track 45.2 -> 30.0 mm, vias 2 -> 1
- net CS_NRF: track 27.3 -> 41.8 mm, vias 1 -> 0
- net CE_NRF: track 31.6 -> 43.5 mm, vias 1 -> 0
- net N$8: track 23.2 -> 11.4 mm
- net N$6: track 5.04 -> 16.7 mm
- net GPS_TX: track 13.7 -> 24.4 mm, vias 1 -> 0
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Other:
- outline, holes or cut-outs redrawn
- board text added: "CE"
- board text added: "CS"
- board text added: "FB SKIRT"
- board text added: "IRQ"
- board text added: "PWR SK CL"
- board text added: "PWR SK OP"
- board text added: "RX"
- board text added: "SCL"
- board text added: "SDA"
- board text added: "TX"
- board text added: "UON"
- board text removed: "CE_NRF"
- board text removed: "CS_NRF"
- board text removed: "USIL_ON"

Commit message: Еще раз проверил все платы и подготовил для производства в Резоните
Parts:
- added DIP-4A: BA159, NEON-BLADE-2023:BA159
- moved C2 2.50 mm to (31.9, 23.8)
- moved C3 2.50 mm to (28.7, 21.0)
- moved INA219 2.50 mm to (31.2, 21.0)
- moved R1 2.50 mm to (33.0, 26.4)
- moved R2 2.50 mm to (30.8, 26.4)
- moved R3 2.50 mm to (31.9, 30.0)
- moved BUTTONS 0.50 mm to (30.7, 11.0)
- turned NRF24L01P to 270 degrees
Connections:
- net N$6: now also DIP-4A.P$2
- net N$8: now also DIP-4A.P$1
Routing:
- net 3V3: track 78.1 -> 103.1 mm, vias 3 -> 5
- net SCK: track 38.0 -> 20.8 mm
- net CE_NRF: track 43.5 -> 30.0 mm
- net NRF_IRQ: track 30.0 -> 40.1 mm
- net GND: track 289.1 -> 297.7 mm, vias 10 -> 9
- net CS_NRF: track 41.8 -> 33.4 mm
- net MOSI: track 40.7 -> 34.8 mm
- net N$8: track 11.4 -> 16.8 mm
- net MISO: track 40.1 -> 34.8 mm
- net N$6: track 16.7 -> 13.3 mm
- net N$4: track 21.6 -> 24.1 mm
- net SDA: track 22.1 -> 19.6 mm
- net SCL: track 22.4 -> 19.9 mm
- net FEEDBACK_SKIRT: track 20.2 -> 19.7 mm
