File: schematics/board/MA_board_2.sch (EAGLE design)
At the start: 16 parts

Commit message: я весь день делал плату с гпской
Parts:
- added J1: MCX-J-P-H-ST-TH1, MCX-J-P-H-ST-TH1:MCX-J-P-H-ST-TH1
- added J2: U.FL-R-SMT-1_10_, U.FL-R-SMT-1_10_:U.FL-R-SMT-1_10_
- added LED1, LED2: (no value), led:LEDSML0603
- added R4, R5: 2k, rcl:R-EU_R0603
- added U$5: GPS, cansat-lib:GPS
- C1: value 100NF -> 100nF
- R1, R2: value 100om -> 100R
- R3: value 0.5om -> R05
Connections:
- new net LED1: LED1.C
- new net LED2: LED2.C
- new net N$2: J2.3, U$4.RF-IN
- new net N$3: J1.1, U$4.ANT
- new net N$7: LED1.A, R4.1
- new net N$9: LED2.A, R5.1
- net 3V3: now also R4.2, R5.2, U$4.LED1, U$4.LED2
- net 5V: now also U$5.UCC
- net FEEDBACK_SKIRT: now also JP4.1, JP7.1
- net GND: now also J1.2, J1.3, J1.4, J1.5, J2.2, JP7.2, U$5.GND; no longer JP3.2
- net GPS_RX: now also U$5.TX
- net GPS_TX: now also U$5.RX
- net MOSI: now also JP1.3; no longer JP1.1
- net POWER_SKIRT_OPEN: now also JP3.2; no longer JP4.1
- net SCK: now also JP1.1; no longer JP1.3
Other:
- moved on the sheet: JP3, JP4, JP5, JP7, U$3, U$4

Commit message: Проверил платы. Исправил некоторые ошибки
Parts:
- removed JP3, JP4, JP5, JP6: (no value), pinhead:PINHD-1X2
- added BATTERY, B_CLOSE, GENERATOR, MOTOR: (no value), pinhead:PINHD-1X2
- added C3: 100nF, rcl:C-EUC0603
- added D1: DIODE-MBR, NEON-BLADE-2023:DIODE-MBR
- C2: value 100NF -> 100nF
- R3: device rcl:R-EU_R2012 -> rcl:R-EU_R2512
- renumbered JP7 to B_OPEN
Connections:
- new net N$8: D1.A, R2.1, R3.2
- net 3V3: now also C3.2; no longer U$4.LED1, U$4.LED2
- net FEEDBACK_SKIRT: now also B_CLOSE.1; no longer JP4.1
- net GND: now also BATTERY.2, B_CLOSE.2, C3.1, GENERATOR.2, J2.1; no longer JP4.2, JP5.2, JP6.2
- net LED1: now also U$4.LED1
- net LED2: now also U$4.LED2
- net N$4: now also GENERATOR.1; no longer JP6.1
- net N$6: now also BATTERY.1, D1.C; no longer JP5.1, R2.1, R3.2
- net POWER_SKIRT_CLOSE: now also MOTOR.1; no longer JP3.1
- net POWER_SKIRT_OPEN: now also MOTOR.2; no longer JP3.2
Other:
- moved on the sheet: JP2

Commit message: Я Данижок, и я тоже сделал плату. А куратор за всех коммитит и выключает компьютеры((
Parts:
- renumbered B_CLOSE to B_CL, B_OPEN to B_OP, U$1 to INA219, U$2 to REF3033, U$4 to AMP

Commit message: Все платы проверены и вроеде бы как готовы к изготовлению!
Parts:
- removed B_CL, B_OP: (no value), pinhead:PINHD-1X2
- added BUTTON-OP, BUTTONS: JST-2-K-S, NEON-BLADE-2023:JST-2-K-S
- added C4: 220uF, NEON-BLADE-2023:ECAPECAP220
- added C6: 100nF, rcl:C-EUC0603
- BATTERY, GENERATOR, MOTOR: value (none) -> JST-2-K-S; device pinhead:PINHD-1X2 -> NEON-BLADE-2023:JST-2-K-S
- D1: value DIODE-MBR -> D-MBR
- JP1, JP2: device pinhead:PINHD-1X8 -> NEON-BLADE-2023:PINHD-1X8-SHORT-PAD
- renumbered U$3 to NRF24L01P
Connections:
- net 5V: now also C4.1, C6.2
- net FEEDBACK_SKIRT: now also BUTTON-OP.2, BUTTONS.1; no longer B_CL.1, B_OP.1
- net GND: now also BUTTON-OP.1, BUTTONS.2, C4.2, C6.1; no longer B_CL.2, B_OP.2
Other:
- moved on the sheet: BATTERY, GENERATOR, MOTOR

Commit message: Еще раз проверил все платы и подготовил для производства в Резоните
Parts:
- added DIP-4A: BA159, NEON-BLADE-2023:BA159
Connections:
- net N$6: now also DIP-4A.C
- net N$8: now also DIP-4A.A
Changed lines of the file:
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@@
 <part name="C6" library="rcl" library_urn="urn:adsk.eagle:library:334" deviceset="C-EU" device="C0603" package3d_urn="urn:adsk.eagle:package:23616/2" value="100nF"/>
 <part name="C4" library="NEON-BLADE-2023" deviceset="ECAP" device="ECAP220" value="220uF"/>
+<part name="DIP-4A" library="NEON-BLADE-2023" deviceset="BA159" device=""/>
 </parts>
 <sheets>
@@
 <attribute name="NAME" x="183.896" y="76.835" size="1.778" layer="95"/>
 <attribute name="VALUE" x="183.896" y="72.009" size="1.778" layer="96"/>
+</instance>
+<instance part="DIP-4A" gate="G$1" x="314.96" y="60.96" smashed="yes">
+<attribute name="NAME" x="312.6486" y="63.6016" size="1.778" layer="95"/>
+<attribute name="VALUE" x="312.3946" y="56.4642" size="1.778" layer="96"/>
 </instance>
 </instances>
@@
 <segment>
 <pinref part="BATTERY" gate="G$1" pin="1"/>
-<wire x1="335.28" y1="71.12" x2="322.58" y2="71.12" width="0.1524" layer="91"/>
+<wire x1="335.28" y1="71.12" x2="325.12" y2="71.12" width="0.1524" layer="91"/>
 <pinref part="D1" gate="G$1" pin="C"/>
+<pinref part="DIP-4A" gate="G$1" pin="C"/>
+<wire x1="325.12" y1="71.12" x2="322.58" y2="71.12" width="0.1524" layer="91"/>
+<wire x1="325.12" y1="71.12" x2="325.12" y2="60.96" width="0.1524" layer="91"/>
+<wire x1="325.12" y1="60.96" x2="317.5" y2="60.96" width="0.1524" layer="91"/>
+<junction x="325.12" y="71.12"/>
 </segment>
 </net>
@@
 <pinref part="R3" gate="G$1" pin="2"/>
 <junction x="302.26" y="71.12"/>
-</segment>
-</net>
+<pinref part="DIP-4A" gate="G$1" pin="A"/>
+<wire x1="302.26" y1="71.12" x2="302.26" y2="60.96" width="0.1524" layer="91"/>
+<wire x1="302.26" y1="60.96" x2="312.42" y2="60.96" width="0.1524" layer="91"/>
+</segment>
+</net>
