File: schematics/board/MA_interface-board.brd (EAGLE design)
At the start: 39 x 26 mm, 28 parts

Commit message: Проверил платы. Исправил некоторые ошибки
Parts:
- added LED8: (no value), led:SML0603
- added R8: 2k, rcl:R0603
- moved R6 4.00 mm to (37.0, 9.50)
- moved U$3 1.50 mm to (2.65, 16.5)
- moved LED7 0.80 mm to (12.3, 21.0)
- moved R7 0.80 mm to (12.3, 24.0)
- moved R5 0.50 mm to (18.7, 9.50)
- moved S1 0.50 mm to (20.0, 22.1)
- moved U$10 0.30 mm to (4.70, 24.5)
Connections:
- new net N$10: LED8.C, R8.1
- net GND: now also R8.2
- net STATE: now also LED8.A

Commit message: Я Тимофей, и я сделал плату. Гыы...
Parts:
- moved JP2 0.22 mm to (37.1, 13.9), turned to 270 degrees
- moved R5 0.10 mm to (18.8, 9.50), turned to 270 degrees
- turned R6 to 270 degrees
Connections:
- removed net DB_RX: JP1.1
- net DBG_RX: now also JP1.1
- net N$7: no longer U$2.P$4
Routing:
- net GND: track 0.00 -> 164.6 mm, vias 0 -> 1
- net 3V3: track 0.00 -> 45.7 mm
- net N$6: track 0.00 -> 36.4 mm, vias 0 -> 1
- net STATE: track 0.00 -> 34.1 mm
- net NRST: track 0.00 -> 31.7 mm, vias 0 -> 2
- net BOTTON_DA_DOWN: track 0.00 -> 27.9 mm, vias 0 -> 1
- net BOTTON_DA_UP: track 0.00 -> 22.5 mm, vias 0 -> 2
- net BOTTON_PAR_DOWN: track 0.00 -> 19.0 mm, vias 0 -> 1
- net BOTTON_PAR_UP: track 0.00 -> 15.6 mm, vias 0 -> 2
- net DBG_RX: track 0.00 -> 14.7 mm
- net BOTTON_SKIRT_CLOSE: track 0.00 -> 14.1 mm, vias 0 -> 1
- net V_BAT: track 0.00 -> 13.8 mm
- net SWD: track 0.00 -> 13.0 mm
- net FEEDBACK_SKIRT: track 0.00 -> 12.7 mm, vias 0 -> 1
- net SDA: track 0.00 -> 11.9 mm
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Other:
- board text added: "100%"
- board text added: "25%"
- board text added: "50%"
- board text added: "75%"
- board text added: "CL"
- board text added: "DA"
- board text added: "DBG"
- board text added: "FLT"
- board text added: "GND"
- board text added: "OP"
- board text added: "POWER"
- board text added: "PWR"
- board text added: "Par"
- board text added: "RST"
- board text added: "ST"
- board text added: "STATE"
- board text added: "SWC/D"
- board text added: "Skirt"
- board text added: "TX/RX"
- board text added: "VB"

Commit message: Все платы проверены и вроеде бы как готовы к изготовлению!
Parts:
- turned LED1 to 90 degrees
- turned LED2 to 90 degrees
- turned LED3 to 90 degrees
- turned LED4 to 90 degrees
Connections:
- net GND: now also LED1.C; no longer R1.1, R2.1, R3.1, R4.1
- net N$7: now also R1.1, R2.1, R3.1, R4.1; no longer LED1.C
Routing:
- net GND: track 164.6 -> 158.6 mm
- net N$4: track 3.48 -> 1.40 mm
- net STATE: track 34.1 -> 35.6 mm
- net N$1: track 5.40 -> 4.12 mm
- net N$2: track 5.40 -> 4.12 mm
- net N$3: track 5.40 -> 4.12 mm
- net N$7: track 11.6 -> 12.3 mm
- net NRST: track 31.7 -> 31.0 mm
- added copper zone on layer 1, net GND
- added copper zone on layer 16, net GND

Commit message: Еще раз проверил все платы и подготовил для производства в Резоните
Changed lines of the file:
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@@
 <layers>
 <layer number="1" name="Top" color="4" fill="1" visible="yes" active="yes"/>
+<layer number="2" name="Route2" color="16" fill="1" visible="no" active="yes"/>
+<layer number="3" name="Route3" color="17" fill="1" visible="no" active="yes"/>
+<layer number="4" name="Route4" color="18" fill="1" visible="no" active="yes"/>
+<layer number="5" name="Route5" color="19" fill="1" visible="no" active="yes"/>
+<layer number="6" name="Route6" color="25" fill="1" visible="no" active="yes"/>
+<layer number="7" name="Route7" color="26" fill="1" visible="no" active="yes"/>
+<layer number="8" name="Route8" color="27" fill="1" visible="no" active="yes"/>
+<layer number="9" name="Route9" color="28" fill="1" visible="no" active="yes"/>
+<layer number="10" name="Route10" color="29" fill="1" visible="no" active="yes"/>
+<layer number="11" name="Route11" color="30" fill="1" visible="no" active="yes"/>
+<layer number="12" name="Route12" color="20" fill="1" visible="no" active="yes"/>
+<layer number="13" name="Route13" color="21" fill="1" visible="no" active="yes"/>
+<layer number="14" name="Route14" color="22" fill="1" visible="no" active="yes"/>
+<layer number="15" name="Route15" color="23" fill="1" visible="no" active="yes"/>
 <layer number="16" name="Bottom" color="1" fill="1" visible="yes" active="yes"/>
 <layer number="17" name="Pads" color="2" fill="1" visible="yes" active="yes"/>
@@
 <param name="mdViaViaSameLayer" value="6mil"/>
 <param name="mnLayersViaInSmd" value="2"/>
-<param name="mdCopperDimension" value="0.3mm"/>
+<param name="mdCopperDimension" value="0.25mm"/>
 <param name="mdDrill" value="6mil"/>
 <param name="mdSmdStop" value="0mil"/>
@@
 <wire x1="16.902" y1="14.098" x2="15.69" y2="15.31" width="0.5" layer="1"/>
 <polygon width="0.1524" layer="1">
-<vertex x="-1" y="28"/>
-<vertex x="41.5" y="28"/>
-<vertex x="41.5" y="-2"/>
-<vertex x="-1" y="-2"/>
+<vertex x="-0.2" y="26.2"/>
+<vertex x="39.2" y="26.2"/>
+<vertex x="39.2" y="-0.2"/>
+<vertex x="-0.2" y="-0.2"/>
 </polygon>
 <polygon width="0.1524" layer="16">
-<vertex x="-1.5" y="28.5"/>
-<vertex x="42" y="28.5"/>
-<vertex x="42" y="-2.5"/>
-<vertex x="-1.5" y="-2.5"/>
+<vertex x="-0.4" y="26.4"/>
+<vertex x="39.4" y="26.4"/>
+<vertex x="39.4" y="-0.4"/>
+<vertex x="-0.4" y="-0.4"/>
 </polygon>
 <contactref element="LED1" pad="C"/>
