File: schematics/board/optical_modul.brd (EAGLE design)
At the start: 42 x 55 mm, 5 parts

Commit message: Все платы проверены и вроеде бы как готовы к изготовлению!
Parts:
- JP1: device pinhead:1X06/90 -> pinhead:1X06
- moved JP1 3.80 mm to (8.00, 5.30)
Routing:
- net IO2: track 37.9 -> 19.6 mm
- net IO0: track 50.5 -> 47.7 mm
- net 5V: track 48.0 -> 46.9 mm
- net GND_ESP: track 76.4 -> 75.6 mm
Changed lines of the file:
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@@
 <?xml version="1.0" encoding="utf-8"?>
 <!DOCTYPE eagle SYSTEM "eagle.dtd">
-<eagle version="9.6.2">
+<eagle version="9.4.2">
 <drawing>
 <settings>
-<setting alwaysvectorfont="no"/>
+<setting alwaysvectorfont="yes"/>
 <setting verticaltext="up"/>
 </settings>
-<grid distance="0.5" unitdist="mm" unit="mm" style="lines" multiple="1" display="no" altdistance="5" altunitdist="mil" altunit="mil"/>
+<grid distance="0.5" unitdist="mm" unit="mm" style="lines" multiple="1" display="no" altdistance="0.1" altunitdist="mm" altunit="mm"/>
 <layers>
 <layer number="1" name="Top" color="4" fill="1" visible="yes" active="yes"/>
@@
 <attribute name="NAME" x="0.68" y="23.84" size="1.27" layer="25" rot="R90"/>
 </element>
-<element name="JP1" library="pinhead" library_urn="urn:adsk.eagle:library:325" package="1X06/90" package3d_urn="urn:adsk.eagle:package:22475/2" value="" x="8" y="1.5" smashed="yes" rot="MR180">
-<attribute name="NAME" x="-0.255" y="5.31" size="1.27" layer="26" ratio="10" rot="MR270"/>
-<attribute name="POPULARITY" value="10" x="8" y="1.5" size="1.778" layer="28" font="vector" rot="MR180" display="off"/>
-<attribute name="VALUE" x="17.525" y="5.31" size="1.27" layer="28" rot="MR270"/>
+<element name="JP1" library="pinhead" library_urn="urn:adsk.eagle:library:325" package="1X06" package3d_urn="urn:adsk.eagle:package:22472/2" value="" x="8" y="5.3" smashed="yes" rot="MR180">
+<attribute name="NAME" x="-0.255" y="9.11" size="1.27" layer="26" ratio="10" rot="MR270"/>
+<attribute name="POPULARITY" value="79" x="8" y="5.3" size="1.778" layer="28" font="vector" rot="MR180" display="off"/>
+<attribute name="VALUE" x="17.525" y="9.11" size="1.27" layer="28" rot="MR270"/>
 </element>
 </elements>
@@
 <contactref element="JP1" pad="1"/>
 <wire x1="22.5" y1="5" x2="22.5" y2="5.05" width="0" layer="19" extent="1-1"/>
-<wire x1="1.65" y1="5.31" x2="1.65" y2="3.35" width="0.5" layer="16"/>
-<wire x1="1.65" y1="3.35" x2="3" y2="2" width="0.5" layer="16"/>
-<wire x1="3" y1="2" x2="19.5" y2="2" width="0.5" layer="16"/>
+<wire x1="5" y1="2" x2="1.7" y2="5.3" width="0.5" layer="16"/>
+<wire x1="1.65" y1="5.3" x2="1.7" y2="5.3" width="0.5" layer="16"/>
+<wire x1="5" y1="2" x2="19.5" y2="2" width="0.5" layer="16"/>
 <wire x1="19.5" y1="2" x2="22.5" y2="5" width="0.5" layer="16"/>
 </signal>
@@
 <wire x1="20.5" y1="5.4242625" x2="10.5" y2="15.4242625" width="0.2" layer="1"/>
 <contactref element="JP1" pad="2"/>
-<wire x1="4.19" y1="5.31" x2="6.8" y2="2.7" width="0.5" layer="16"/>
+<wire x1="4.19" y1="5.3" x2="6.79" y2="2.7" width="0.5" layer="16"/>
 <wire x1="18.2" y1="2.7" x2="20.5" y2="5" width="0.5" layer="16"/>
-<wire x1="6.8" y1="2.7" x2="18.2" y2="2.7" width="0.5" layer="16"/>
+<wire x1="6.79" y1="2.7" x2="18.2" y2="2.7" width="0.5" layer="16"/>
 <wire x1="20.5" y1="5" x2="20.5" y2="5.05" width="0" layer="19" extent="1-16"/>
 </signal>
@@
 <wire x1="19.5" y1="3.9" x2="19.5" y2="5.05" width="0.5" layer="1"/>
 <wire x1="26.95" y1="4.45" x2="37.5" y2="15" width="0.5" layer="1"/>
-<wire x1="18.64" y1="44.93" x2="18.64" y2="43.5" width="0.5" layer="1"/>
-<wire x1="18.64" y1="43.5" x2="28.8" y2="43.5" width="0.5" layer="1"/>
+<wire x1="28.8" y1="43.5" x2="32" y2="43.5" width="0.5" layer="1"/>
 <wire x1="28.8" y1="44.9742625" x2="28.8" y2="43.5" width="0.5" layer="1"/>
-<wire x1="28.8" y1="43.5" x2="33.8" y2="38.5" width="0.5" layer="1"/>
-<wire x1="33.8" y1="38.5" x2="37" y2="38.5" width="0.5" layer="1"/>
-<wire x1="37.5" y1="38" x2="37" y2="38.5" width="0.5" layer="1"/>
+<wire x1="32" y1="43.5" x2="37.5" y2="38" width="0.5" layer="1"/>
 <wire x1="37.5" y1="15" x2="37.5" y2="23.5" width="0.5" layer="1"/>
 <wire x1="37.5" y1="23.5" x2="37.5" y2="38" width="0.5" layer="1"/>
 <wire x1="33.88" y1="22.07" x2="35.31" y2="23.5" width="0.5" layer="1"/>
 <wire x1="35.31" y1="23.5" x2="37.5" y2="23.5" width="0.5" layer="1"/>
+<wire x1="18.64" y1="44.93" x2="20.07" y2="43.5" width="0.5" layer="1"/>
+<wire x1="20.07" y1="43.5" x2="28.8" y2="43.5" width="0.5" layer="1"/>
 </signal>
 <signal name="U0T">
 <contactref element="JP1" pad="3"/>
 <contactref element="U$4" pad="P$15"/>
-<wire x1="6.73" y1="5.31" x2="6.73" y2="18.73" width="0.2" layer="16"/>
-<wire x1="6.73" y1="18.73" x2="21.5" y2="33.5" width="0.2" layer="16"/>
-<wire x1="21.5" y1="33.5" x2="21.5" y2="44.61" width="0.2" layer="16"/>
-<wire x1="21.5" y1="44.61" x2="21.18" y2="44.93" width="0.2" layer="16"/>
+<wire x1="6.73" y1="5.3" x2="6.73" y2="18.73" width="0.2" layer="16"/>
+<wire x1="6.73" y1="18.73" x2="21.2" y2="33.2" width="0.2" layer="16"/>
+<wire x1="21.2" y1="33.2" x2="21.2" y2="44.91" width="0.2" layer="16"/>
+<wire x1="21.2" y1="44.91" x2="21.18" y2="44.93" width="0.2" layer="16"/>
 </signal>
 <signal name="U0R">
 <contactref element="JP1" pad="4"/>
 <contactref element="U$4" pad="P$14"/>
-<wire x1="9.27" y1="5.31" x2="9.27" y2="18.27" width="0.2" layer="16"/>
-<wire x1="9.27" y1="18.27" x2="24" y2="33" width="0.2" layer="16"/>
-<wire x1="24" y1="33" x2="24" y2="44.65" width="0.2" layer="16"/>
-<wire x1="24" y1="44.65" x2="23.72" y2="44.93" width="0.2" layer="16"/>
+<wire x1="9.27" y1="5.3" x2="9.27" y2="18.27" width="0.2" layer="16"/>
+<wire x1="9.27" y1="18.27" x2="23.7" y2="32.7" width="0.2" layer="16"/>
+<wire x1="23.72" y1="44.93" x2="23.7" y2="44.91" width="0.2" layer="16"/>
+<wire x1="23.7" y1="44.91" x2="23.7" y2="32.7" width="0.2" layer="16"/>
 </signal>
 <signal name="IO0">
 <contactref element="JP1" pad="5"/>
 <contactref element="U$4" pad="P$11"/>
-<wire x1="11.81" y1="5.31" x2="11.81" y2="17.31" width="0.2" layer="16"/>
-<wire x1="27" y1="32.5" x2="27" y2="42.5" width="0.2" layer="16"/>
-<wire x1="27" y1="42.5" x2="31.5" y2="42.5" width="0.2" layer="16"/>
-<wire x1="31.5" y1="42.5" x2="31.5" y2="44.77" width="0.2" layer="16"/>
-<wire x1="31.5" y1="44.77" x2="31.34" y2="44.93" width="0.2" layer="16"/>
-<wire x1="11.81" y1="17.31" x2="27" y2="32.5" width="0.2" layer="16"/>
+<wire x1="11.81" y1="5.3" x2="11.81" y2="17.31" width="0.2" layer="16"/>
+<wire x1="26" y1="31.5" x2="11.81" y2="17.31" width="0.2" layer="16"/>
+<wire x1="31.34" y1="44.93" x2="26" y2="39.59" width="0.2" layer="16"/>
+<wire x1="26" y1="39.59" x2="26" y2="31.5" width="0.2" layer="16"/>
 </signal>
 <signal name="IO2">
 <contactref element="JP1" pad="6"/>
 <contactref element="U$4" pad="P$7"/>
-<wire x1="14.35" y1="5.31" x2="19.04" y2="10" width="0.2" layer="16"/>
-<wire x1="19.04" y1="10" x2="26.5" y2="10" width="0.2" layer="16"/>
-<wire x1="26.5" y1="10" x2="31.5" y2="15" width="0.2" layer="16"/>
-<wire x1="31.5" y1="15" x2="31.5" y2="18" width="0.2" layer="16"/>
-<wire x1="31.5" y1="18" x2="30" y2="19.5" width="0.2" layer="16"/>
-<wire x1="30" y1="19.5" x2="21" y2="19.5" width="0.2" layer="16"/>
-<wire x1="21" y1="19.5" x2="21" y2="21.89" width="0.2" layer="16"/>
-<wire x1="21" y1="21.89" x2="21.18" y2="22.07" width="0.2" layer="16"/>
+<wire x1="14.35" y1="5.85" x2="14.35" y2="5.3" width="0.2" layer="16"/>
+<wire x1="21.18" y1="22.07" x2="21.18" y2="22.0290375" width="0.2" layer="16"/>
+<wire x1="21.18" y1="22.0290375" x2="18.5" y2="19.3490375" width="0.2" layer="16"/>
+<wire x1="18.5" y1="19.3490375" x2="18.5" y2="10" width="0.2" layer="16"/>
+<wire x1="18.5" y1="10" x2="14.35" y2="5.85" width="0.2" layer="16"/>
 </signal>
 </signals>

Commit message: Еще раз проверил все платы и подготовил для производства в Резоните
Parts:
- renumbered JP1 to DEBAG, U$4 to ESP32-CAM
Connections:
- net GND: no longer DEBAG.2
- net GND_ESP: now also DEBAG.2
Routing:
- net GND: track 77.3 -> 59.0 mm
- net GND_ESP: track 75.6 -> 92.3 mm, vias 0 -> 1
- net 5V: track 46.9 -> 51.1 mm, vias 0 -> 1
- net FEEDBACK_DA: track 59.7 -> 55.8 mm
- added copper zone on layer 1, net GND_ESP
- added copper zone on layer 16, net GND_ESP
Other:
- board text added: "(GND)"
- board text added: "5V"
- board text added: "GND-ESP"
- board text added: "IO0"
- board text added: "IO2"
- board text added: "U0R"
- board text added: "U0T"
