File: schematics/board/Cansat-2023-1.brd (EAGLE design)
At the start: 68 x 75.2 mm, 79 parts, among them Q24 Q24

Commit message: Еще раз проверил все платы и подготовил для производства в Резоните
Parts:
- added -BAT+, JP8, PWR-SW: (no value), pinhead:1X02
- added 1, 2, 3: 4-PIN, CanCubeSat:4PINHEADERSMD
- added 3V1, 5V1, PPS, SCK, VBAT: (no value), led:CHIP-LED0603
- added A, B: 24-PIN, CanCubeSat:24PINHEADERSMD
- added AMP: XQ-02A, NEON-BLADE-2023:XQ-02A
- added BATTERY, BUTTON-OP, BUTTONS, GENERATOR, MOTOR: JST-2-K-S, NEON-BLADE-2023:B2B-PH-K-S
- added C12, C13, C14, C15: 100nF, rcl:C0603
- added C16: 220uF, NEON-BLADE-2023:ECAP220-CMD
- added C17, C18, C19, C20: 10µF, rcl:C1206
- added CHRG: (no value), pinhead:1X02/90
- added D1: D-MBR, NEON-BLADE-2023:SOD123
- added DEBAG: (no value), pinhead:1X06
- added DIP-4A: BA159, NEON-BLADE-2023:BA159
- added ESP32-CAM: ESP32-CAM, NEON-BLADE-2023:ESP32-CAM
- added INA219: INA219AID, NEON-BLADE-2023:SOT23-8
- added J1: MCX-J-P-H-ST-TH1, MCX-J-P-H-ST-TH1:MCXJPHSTTH1
- added J2: U.FL-R-SMT-1_10_, U.FL-R-SMT-1_10_:U.FL-R-SMT-1(10)
- added JP10: (no value), pinhead:2X02
- added JP5: (no value), pinhead:1X04
- added JP9: (no value), pinhead:2X10
- added LED1, LED10, LED2, LED3, LED4, LED5, LED6, LED7, LED8, LED9: (no value), led:SML0603
- added PWR_BL_SW: (no value), jumper:SJ_2
- added R38, R39, R57: 100R, rcl:R0603
- added R40, R41, R47, R48, R50, R52, R54: 2k, rcl:R0603
- added R42: R05, rcl:R2512
- added R43, R44, R45, R46, R51, R53, R58: 1k, rcl:R0603
- added R49: 5K1, rcl:R0603
- added R55: (no value), rcl:R0603
- added R56: 5k1, rcl:R0603
- added REF3033: REF3033, NEON-BLADE-2023:SOT23-3
- added S1: (no value), cansat-lib:UNICS-SWITCH
- added U$1: FCC-CONNECT-6P, NEON-BLADE-2023:FFC-CONNECT-6P-SMD
- added U$10, U$11, U$13, U$14, U$15, U$2, U$3, U$6, U$7, U$9: BTN_VERY_SMALL, NEON-BLADE-2023:BTN_VERY_SMALL
- added U$18: MSS12D01, NEON-BLADE-2023:MSS12D01
- added U$4: BME280BME280-PINS-ONLY, NEON-BLADE-2023:BME280-PINS-ONLY
- added U$5: GPS, cansat-lib:GPS
Connections:
- new net +3V3: A.23, B.23, R53.2, R55.2, R57.2
- new net +5V: A.9, B.9, PWR_BL_SW.1, R52.2
- new net 3V1: C14.2, INA219.4, R40.2, R41.2, REF3033.2
- new net 3V2: JP9.15, R47.2, R48.2, U$18.P$2, U$4.P$1
- new net 5V1: AMP.P$5, C12.1, C15.2, C16.P$1, REF3033.1, U$5.UCC
- new net 5V2: DEBAG.1, ESP32-CAM.P$1, U$1.P$5, U$1.P$6
- new net BOTTON_DA_DOWN1: JP9.9, U$9.P$1, U$9.P$2
- new net BOTTON_DA_UP1: JP9.7, U$10.P$1, U$10.P$2
- new net BOTTON_PAR_DOWN1: JP9.12, U$11.P$1, U$11.P$2
- new net BOTTON_PAR_UP1: JP9.10, U$13.P$1, U$13.P$2
- new net BOTTON_SKIRT_CLOSE1: JP9.8, U$15.P$1, U$15.P$2
- new net BOTTON_SKIRT_OPEN1: JP9.6, U$14.P$1, U$14.P$2
- new net DBG_RX1: JP5.1, JP9.18
- new net DBG_TX1: JP5.2, JP9.20
- new net FEEDBACK_DA1: U$1.P$4, U$2.P$1, U$2.P$2, U$3.P$1, U$3.P$2
- new net FEEDBACK_DA2: JP9.4, LED8.C
- new net FEEDBACK_SKIRT1: BUTTON-OP.2, BUTTONS.1
- new net FEEDBACK_SKIRT2: JP9.3, LED7.C
- new net GND1: AMP.P$1, AMP.P$10, AMP.P$12, AMP.P$13, AMP.P$2, AMP.P$4, BATTERY.2, BUTTON-OP.1, BUTTONS.2, C12.2, C14.1, C15.1, C16.P$2, GENERATOR.2, INA219.3, INA219.7, INA219.8, J1.2, J1.3, J1.4, J1.5, J2.1, J2.2, REF3033.3, U$5.GND
- new net GND2: U$1.P$3, U$2.P$3, U$2.P$4, U$3.P$3, U$3.P$4
- new net GND3: JP8.2, JP9.13, LED3.C, R49.2, R50.2, U$10.P$3, U$10.P$4, U$11.P$3, U$11.P$4, U$13.P$3, U$13.P$4, U$14.P$3, U$14.P$4, U$15.P$3, U$15.P$4, U$18.P$3, U$4.P$2, U$7.P$3, U$7.P$4, U$9.P$3, U$9.P$4
- new net GND4: 1.3, 2.3, 3.3, 3V1.C, 5V1.C, A.10, A.16, A.2, A.24, B.10, B.16, B.2, B.24, C18.1, C19.1, C20.1, JP10.1, PPS.C, PWR-SW.1, R56.1, SCK.C, VBAT.C
- new net GND_ESP1: DEBAG.2, ESP32-CAM.P$12, ESP32-CAM.P$16, ESP32-CAM.P$2, U$1.P$1, U$1.P$2
- new net GPS_RX1: U$5.TX
- new net GPS_TX1: U$5.RX
- new net IO0: DEBAG.5, ESP32-CAM.P$11
- new net IO2: DEBAG.6, ESP32-CAM.P$7
- new net LED1: AMP.P$8, LED1.C
- new net LED2: AMP.P$9, LED2.C
- new net N$15: C13.1, INA219.1, R38.2
- new net N$16: C13.2, INA219.2, R39.2
- new net N$18: BATTERY.1, D1.C, DIP-4A.P$2
- new net N$19: GENERATOR.1, R38.1, R42.1
- new net N$21: AMP.P$3, J2.3
- new net N$22: AMP.P$11, J1.1
- new net N$23: LED1.A, R40.1
- new net N$24: LED2.A, R41.1
- new net N$25: D1.A, DIP-4A.P$1, R39.1, R42.2
- new net N$26: LED3.A, LED4.C, R43.2
- new net N$27: LED4.A, LED5.C, R44.2
- new net N$28: LED5.A, LED6.C, R45.2
- new net N$29: LED6.A, R46.2
- new net N$30: JP8.1, S1.1, U$6.P$1, U$6.P$2
- new net N$31: LED7.A, R47.1
- new net N$32: LED8.A, R48.1
- new net N$33: LED9.C, R49.1
- new net N$34: LED10.C, R50.1
- new net N$35: R43.1, R44.1, R45.1, R46.1, U$6.P$3
- new net N$38: R51.1, SCK.A
- new net N$39: 5V1.A, R52.1
- new net N$40: 3V1.A, R53.1
- new net N$41: PPS.A, R54.1
- new net N$42: -BAT+.2, C17.1, CHRG.2, PWR-SW.2
- new net N$43: JP10.4, R57.1
- new net N$44: R58.1, VBAT.A
- new net NRST1: JP9.5, U$7.P$1, U$7.P$2
- new net PHOT: B.4, JP10.2, R55.1
- new net POWER_SKIRT_CLOSE1: MOTOR.1
- new net POWER_SKIRT_OPEN1: MOTOR.2
- new net PPS: A.13, R54.2
- new net SCL1: INA219.5
- new net SCL2: JP9.16, U$4.P$3
- new net SCL3: 1.1, 2.1, 3.1, B.19, R51.2
- new net SDA1: INA219.6
- new net SDA2: JP9.14, U$4.P$4
- new net SDA3: 1.2, 2.2, 3.2, B.20
- new net ST-SW: B.1, JP10.3, R56.2
- new net STATE1: JP9.1, LED10.A, U$18.P$1
- new net SWC: JP5.4, JP9.19
- new net SWD: JP5.3, JP9.17
- new net U0R: DEBAG.4, ESP32-CAM.P$14
- new net U0T: DEBAG.3, ESP32-CAM.P$15
- new net USIL_ON1: AMP.P$7
- new net V+: -BAT+.1, A.15, B.15, C17.2, CHRG.1, PWR_BL_SW.3, R58.2
- new net VCC: 1.4, 2.4, 3.4, C18.2, C19.2, C20.2, PWR_BL_SW.2
- new net V_BAT1: JP9.11, LED9.A, S1.2
Routing:
- net GND1: track 0.00 -> 237.3 mm, vias 0 -> 9
- net GND3: track 0.00 -> 158.6 mm, vias 0 -> 1
- net GND_ESP1: track 0.00 -> 92.3 mm, vias 0 -> 1
- net 5V1: track 0.00 -> 84.4 mm
- net SDA3: track 0.00 -> 77.1 mm, vias 0 -> 5
- net SCL3: track 0.00 -> 73.6 mm, vias 0 -> 1
- net GND2: track 0.00 -> 59.0 mm, vias 0 -> 2
- net FEEDBACK_DA1: track 0.00 -> 55.8 mm, vias 0 -> 3
- net USIL_ON1: track 0.00 -> 53.1 mm
- net +5V: track 0.00 -> 51.6 mm
- net 5V2: track 0.00 -> 51.1 mm, vias 0 -> 1
- net IO0: track 0.00 -> 47.7 mm
- net 3V2: track 0.00 -> 45.7 mm
- net U0T: track 0.00 -> 45.6 mm
- net U0R: track 0.00 -> 45.6 mm
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- added copper zone on layer 16, net +3V3
- added copper zone on layer 1, net GND1
- added copper zone on layer 1, net GND3
- added copper zone on layer 16, net GND3
- added copper zone on layer 1, net GND4
- added copper zone on layer 1, net GND_ESP1
- added copper zone on layer 16, net GND_ESP1
- added copper zone on layer 16, net V+
- added copper zone on layer 16, net VCC
Other:
- board size 68 x 75.2 mm -> 119 x 134 mm
- board text added: "(GND)"
- board text added: "+"
- board text added: "-"
- board text added: "100%"
- board text added: "25%"
- board text added: "50%"
- board text added: "75%"
- board text added: "ANT"
- board text added: "CE"
- board text added: "CL"
- board text added: "CS"
- board text added: "DA"
- board text added: "DBG"
- board text added: "FB SKIRT"
- board text added: "FLT"
- board text added: "GND-ESP"
- board text added: "IO0"
- board text added: "IO2"
- board text added: "IRQ"
- board text added: "OP"
- board text added: "POWER"
- board text added: "PWR"
- board text added: "PWR SK CL"
- board text added: "PWR SK OP"
- board text added: "Par"
- board text added: "RST"
- board text added: "RX"
- board text added: "ST"
- board text added: "SWC/D"
- board text added: "Skirt"
- board text added: "TX"
- board text added: "TX/RX"
- board text added: "U0R"
- board text added: "U0T"
- board text added: "UON"
- board text added: "VB"
- board text added: "Vbat"
- board text added: "nRF24"

Commit message: Комплекты плат, которые были отправлены на производство (кроме платы ДА)
Parts:
- added JP11, JP12: (no value), NEON-BLADE-2023:1X08
- added NRF24L01P: NRF24L01_ML01SP4, NEON-BLADE-2023:NRF24L01_ML01SP4
Connections:
- new net CE_NRF1: JP11.5, NRF24L01P.P$2
- new net CS_NRF1: JP11.4, NRF24L01P.P$3
- new net MISO1: JP11.2, NRF24L01P.P$6
- new net MOSI1: JP11.3, NRF24L01P.P$5
- new net NRF_IRQ1: JP12.5, NRF24L01P.P$7
- new net SCK1: JP11.1, NRF24L01P.P$4
- net 3V1: now also NRF24L01P.P$1
- net 5V1: now also JP11.8
- net FEEDBACK_SKIRT1: now also JP12.6
- net GND1: now also JP11.7, NRF24L01P.P$8
- net GPS_RX1: now also JP12.1
- net GPS_TX1: now also JP12.2
- net POWER_SKIRT_CLOSE1: now also JP12.8
- net POWER_SKIRT_OPEN1: now also JP12.7
- net SCL1: now also JP12.4
- net SDA1: now also JP12.3
- net USIL_ON1: now also JP11.6
Routing:
- net 3V1: track 28.5 -> 103.1 mm
- net GND1: track 237.3 -> 297.7 mm
- net MISO1: track 0.00 -> 34.8 mm
- net MOSI1: track 0.00 -> 34.8 mm
- net CS_NRF1: track 0.00 -> 33.4 mm
- net CE_NRF1: track 0.00 -> 30.0 mm
- net POWER_SKIRT_CLOSE1: track 0.00 -> 27.0 mm
- net POWER_SKIRT_OPEN1: track 0.00 -> 21.0 mm
- net SCK1: track 3.91 -> 20.8 mm
- net NRF_IRQ1: track 37.1 -> 40.1 mm
- added copper zone on layer 16, net GND1
