File: schematics/board/Cansat-2023-2.brd (EAGLE design)
At the start: 71.7 x 128.4 mm, 233 parts, among them P0102BL P0102BL, P0102BL1 P0102BL, P0102BL2 P0102BL

Commit message: Комплекты плат, которые были отправлены на производство (кроме платы ДА)
Parts:
- R10: value 1k -> 1k*2
- moved SI3 0.22 mm to (26.5, 38.7)
Other:
- board text added: "GND"
- board text added: "RES"
- board text added: "SCL"
- board text added: "SDA"
- board text added: "VCC"
- board text removed: "Middle board This side up By ATLAS++ Korolyov, TSNIIMASH"
