File: schematics/board/Cansat-2023-3.brd (EAGLE design)
At the start: 114 x 82 mm, 66 parts, among them Q24 Q24

Commit message: Комплекты плат, которые были отправлены на производство (кроме платы ДА)
Parts:
- moved R7 2.02 mm to (52.2, 47.9)
- moved BUZZER 2.00 mm to (58.0, 41.2)
- moved MICROSD 2.00 mm to (35.0, 33.5)
- moved R8 1.22 mm to (54.3, 47.9), turned to 90 degrees
- moved SI2301 1.17 mm to (60.6, 48.0)
Routing:
- net 5V: track 193.6 -> 190.5 mm
- net GND: track 283.8 -> 286.4 mm
- net SDIO_DAT3: track 15.4 -> 17.6 mm
- net SDIO_DAT2: track 13.0 -> 15.0 mm
- net SDIO_DAT1: track 39.1 -> 41.1 mm
- net SDIO_DAT0: track 37.3 -> 39.3 mm
- net SDIO_CK: track 18.2 -> 20.2 mm
- net N$20: track 5.80 -> 7.49 mm
- net CS_LIS: track 40.9 -> 42.5 mm
- net CS_LSM: track 86.9 -> 85.8 mm
- net SDIO_CMD: track 19.5 -> 18.4 mm
- net SDA: track 27.8 -> 28.3 mm
- net SCL: track 27.6 -> 28.1 mm
- added copper zone on layer 1, net P1
- added copper zone on layer 16, net P1
- added copper zone on layer 1, net P3
- added copper zone on layer 16, net P3
- added copper zone on layer 1, net P5
- added copper zone on layer 16, net P5
- added copper zone on layer 1, net SP-
- added copper zone on layer 16, net SP-
