File: schematics/board/DA.brd (EAGLE design)
At the start: 82 x 82 mm, 48 parts, among them Q24 Q24

Commit message: Еще раз проверил все платы и подготовил для производства в Резоните
Parts:
- moved LIS3MDL 0.10 mm to (23.2, 20.0)
Routing:
- net 5V: track 191.3 -> 193.6 mm
- net CS_NRF: track 97.8 -> 98.6 mm
- net GPS_RX: track 77.9 -> 78.3 mm, vias 1 -> 3

Commit message: Комплекты плат, которые были отправлены на производство (кроме платы ДА)
Parts:
- moved R7 2.02 mm to (20.2, 47.9)
- moved BUZZER 2.00 mm to (26.0, 41.2)
- moved MICROSD 2.00 mm to (3.00, 33.5)
- moved R8 1.22 mm to (22.3, 47.9), turned to 90 degrees
- moved SI2301 1.17 mm to (28.6, 48.0)
Routing:
- net 5V: track 193.6 -> 190.5 mm
- net GND: track 283.8 -> 286.4 mm
- net SDIO_DAT3: track 15.4 -> 17.6 mm
- net SDIO_DAT2: track 13.0 -> 15.0 mm
- net SDIO_DAT1: track 39.1 -> 41.1 mm
- net SDIO_DAT0: track 37.3 -> 39.3 mm
- net SDIO_CK: track 18.2 -> 20.2 mm
- net N$20: track 5.80 -> 7.49 mm
- net CS_LIS: track 40.9 -> 42.5 mm
- net CS_LSM: track 86.9 -> 85.8 mm
- net SDIO_CMD: track 19.5 -> 18.4 mm
- net SDA: track 27.8 -> 28.3 mm
- net SCL: track 27.6 -> 28.1 mm
